File: schematic/Stazione_Meteo.brd (EAGLE design)
At the start: 100 x 75 mm, 28 parts

Commit message: removed diode on power supply inlet
power is +5V, diode drops 0.7V leaving available only 4.3V, not suitable for voltage regulator on NodeMCU
Parts:
- removed D1: 1N4004, diode:DO41-10
Connections:
- removed net N$5: D1.A, X1.1
- net +5V: now also X1.1; no longer D1.C
Routing:
- net +5V: track 186.4 -> 199.4 mm
- net N$5: track 9.00 -> 0.00 mm
Changed lines of the file:
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@@
 <?xml version="1.0" encoding="utf-8"?>
 <!DOCTYPE eagle SYSTEM "eagle.dtd">
-<eagle version="7.7.0">
+<eagle version="7.4.0">
 <drawing>
 <settings>
@@
 <attribute name="VALUE" x="40.2034" y="72.7004" size="1.27" layer="27" ratio="10" rot="R90"/>
 </element>
-<element name="D1" library="diode" package="DO41-10" value="1N4004" x="12.5175" y="61.84125" smashed="yes">
-<attribute name="NAME" x="11.91425" y="63.3335" size="1.27" layer="25" font="vector" ratio="10"/>
-<attribute name="VALUE" x="9.2155" y="59.206" size="1.27" layer="27" font="vector" ratio="10"/>
-</element>
 <element name="S1" library="switch-omron" package="B3F-10XX" value="" x="28.06375" y="69.47625" smashed="yes" rot="R180">
 <attribute name="OC_FARNELL" value="176432" x="28.06375" y="69.47625" size="1.778" layer="27" rot="R180" display="off"/>
@@
 <wire x1="15.08125" y1="17.145" x2="11.43" y2="17.145" width="0.8128" layer="16"/>
 </signal>
-<signal name="N$5">
-<contactref element="X1" pad="1"/>
-<contactref element="D1" pad="A"/>
-<wire x1="15" y1="69.77" x2="15" y2="64.43875" width="0.8128" layer="16"/>
-<wire x1="15" y1="64.43875" x2="17.5975" y2="61.84125" width="0.8128" layer="16"/>
-</signal>
 <signal name="+5V">
 <contactref element="C6" pad="+"/>
-<contactref element="D1" pad="C"/>
 <contactref element="C1" pad="1"/>
 <contactref element="U$1" pad="VIN"/>
@@
 <wire x1="17.145" y1="12.065" x2="19.05" y2="13.97" width="0.8128" layer="16"/>
 <contactref element="C5" pad="1"/>
-<wire x1="7.4375" y1="61.84125" x2="7.4375" y2="58.7075" width="0.8128" layer="16"/>
-<wire x1="7.4375" y1="58.7075" x2="6.115" y2="57.385" width="0.8128" layer="16"/>
-<wire x1="6.115" y1="57.385" x2="5.1" y2="56.37" width="0.8128" layer="16"/>
 <wire x1="6.35" y1="47.3075" x2="6.35" y2="49.53" width="0.8128" layer="16"/>
 <wire x1="6.35" y1="49.53" x2="7.62" y2="50.8" width="0.8128" layer="16"/>
 <wire x1="7.62" y1="50.8" x2="7.62" y2="55.88" width="0.8128" layer="16"/>
-<wire x1="7.62" y1="55.88" x2="6.115" y2="57.385" width="0.8128" layer="16"/>
 <wire x1="6.35" y1="19.05" x2="9.36625" y2="16.03375" width="0.8128" layer="16"/>
 <wire x1="9.36625" y1="16.03375" x2="9.36625" y2="12.365" width="0.8128" layer="16"/>
@@
 <wire x1="9.36625" y1="27.305" x2="9.36625" y2="31.115" width="0.8128" layer="16"/>
 <wire x1="9.36625" y1="31.115" x2="4.683125" y2="35.798125" width="0.8128" layer="16"/>
+<contactref element="X1" pad="1"/>
+<wire x1="5.1" y1="56.37" x2="7.13" y2="56.37" width="0.8128" layer="16"/>
+<wire x1="7.13" y1="56.37" x2="7.62" y2="55.88" width="0.8128" layer="16"/>
+<wire x1="7.13" y1="56.37" x2="7.13" y2="60.47" width="0.8128" layer="16"/>
+<wire x1="7.13" y1="60.47" x2="8.89" y2="62.23" width="0.8128" layer="16"/>
+<wire x1="8.89" y1="62.23" x2="12.6746" y2="62.23" width="0.8128" layer="16"/>
+<wire x1="12.6746" y1="62.23" x2="15.0368" y2="64.5922" width="0.8128" layer="16"/>
+<wire x1="15.0368" y1="64.5922" x2="15.0368" y2="69.7332" width="0.8128" layer="16"/>
+<wire x1="15.0368" y1="69.7332" x2="15" y2="69.77" width="0.8128" layer="16"/>
 </signal>
 <signal name="N$9">
