File: schematic/Stazione_Meteo.sch (EAGLE design)
At the start: 28 parts

Commit message: removed diode on power supply inlet
power is +5V, diode drops 0.7V leaving available only 4.3V, not suitable for voltage regulator on NodeMCU
Parts:
- removed D1: 1N4004, diode:1N4004
Connections:
- removed net N$5: D1.A, X1-1.KL
- net +5V: now also X1-1.KL; no longer D1.C
Changed lines of the file:
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@@
 <?xml version="1.0" encoding="utf-8"?>
 <!DOCTYPE eagle SYSTEM "eagle.dtd">
-<eagle version="7.7.0">
+<eagle version="7.4.0">
 <drawing>
 <settings>
@@
 <part name="R3" library="rcl" deviceset="R-EU_" device="0204/7" value="100R"/>
 <part name="LED1" library="led" deviceset="LED" device="5MM"/>
-<part name="D1" library="diode" deviceset="1N4004" device=""/>
 <part name="GND6" library="supply1" deviceset="GND" device=""/>
 <part name="S1" library="switch-omron" deviceset="10-XX" device=""/>
@@
 <instance part="R3" gate="G$1" x="40.64" y="7.62" rot="R90"/>
 <instance part="LED1" gate="G$1" x="45.72" y="15.24" rot="R90"/>
-<instance part="D1" gate="1" x="-22.86" y="-63.5"/>
 <instance part="GND6" gate="1" x="55.88" y="7.62"/>
 <instance part="S1" gate="1" x="-27.94" y="-30.48" rot="R270"/>
@@
 </segment>
 </net>
-<net name="N$5" class="0">
-<segment>
-<pinref part="X1" gate="-1" pin="KL"/>
-<pinref part="D1" gate="1" pin="A"/>
-<wire x1="-30.48" y1="-63.5" x2="-25.4" y2="-63.5" width="0.1524" layer="91"/>
-</segment>
-</net>
 <net name="+5V" class="0">
 <segment>
-<pinref part="D1" gate="1" pin="C"/>
-<wire x1="-20.32" y1="-63.5" x2="-7.62" y2="-63.5" width="0.1524" layer="91"/>
+<wire x1="-30.48" y1="-63.5" x2="-7.62" y2="-63.5" width="0.1524" layer="91"/>
 <pinref part="C6" gate="G$1" pin="+"/>
 <wire x1="-7.62" y1="-63.5" x2="0" y2="-63.5" width="0.1524" layer="91"/>
@@
 <wire x1="0" y1="-66.04" x2="0" y2="-63.5" width="0.1524" layer="91"/>
 <junction x="0" y="-63.5"/>
-</segment>
-<segment>
+<pinref part="X1" gate="-1" pin="KL"/>
+</segment>
+<segment>
